File: PCB/LinKey.kicad_sch (KiCad schematic)
At the start: 1 part

Commit message: Release PCB v1
Parts:
- added C1: 2,2u, Capacitor_SMD:C_0805_2012Metric_Pad1.18x1.45mm_HandSolder, symbol Device:C
- added C2: 1F, Capacitor_THT:CP_Radial_D8.0mm_P3.50mm, symbol Device:C_Polarized
- added C3, C6, C7: 22u, Capacitor_SMD:C_1206_3216Metric_Pad1.33x1.80mm_HandSolder, symbol Device:C
- added C4, C8: 100n, Capacitor_SMD:C_0603_1608Metric_Pad1.08x0.95mm_HandSolder, symbol Device:C
- added C5: 175p, Capacitor_SMD:C_0603_1608Metric_Pad1.08x0.95mm_HandSolder, symbol Device:C
- added D1: BAS_4002A_RPP_E6327, LinKey_Lib_Footprints:BAS4002ARPPE6327, symbol LinKey_Lib_Symbols:BAS_4002A_RPP_E6327
- added D8: LED_RGB, LED_SMD:LED_RGB_5050-6, symbol Device:LED_RGB
- added J2: Conn_01x04, Connector_PinHeader_2.54mm:PinHeader_1x04_P2.54mm_Vertical, symbol Connector_Generic:Conn_01x04
- added L1: 1uH, Inductor_SMD:L_Coilcraft_XAL5030-XXX, symbol Device:L_Iron_Small
- added Q1: MMBT2907ALT1G, Package_TO_SOT_SMD:SOT-23_Handsoldering, symbol Transistor_BJT:MMBTA94
- added Q2: CSD25402Q3A, Package_SON:VSON-8_3.3x3.3mm_P0.65mm_NexFET, symbol Transistor_FET:CSD25402Q3A
- added R1, R2, R3: R, Resistor_SMD:R_0603_1608Metric_Pad0.98x0.95mm_HandSolder, symbol Device:R
- added R10: 18r, Resistor_SMD:R_1206_3216Metric_Pad1.30x1.75mm_HandSolder, symbol Device:R
- added R11: 200r, Resistor_SMD:R_0603_1608Metric_Pad0.98x0.95mm_HandSolder, symbol Device:R
- added R12, R6, R9: 120r, Resistor_SMD:R_0603_1608Metric_Pad0.98x0.95mm_HandSolder, symbol Device:R
- added R13, R15, R5, R7: 10k, Resistor_SMD:R_0603_1608Metric_Pad0.98x0.95mm_HandSolder, symbol Device:R
- added R14: 2k, Resistor_SMD:R_0603_1608Metric_Pad0.98x0.95mm_HandSolder, symbol Device:R
- added R16, R18: 100k, Resistor_SMD:R_0603_1608Metric_Pad0.98x0.95mm_HandSolder, symbol Device:R
- added R17: 453k, Resistor_SMD:R_0603_1608Metric_Pad0.98x0.95mm_HandSolder, symbol Device:R
- added R4: 470r, Resistor_SMD:R_0603_1608Metric_Pad0.98x0.95mm_HandSolder, symbol Device:R
- added R8: 330r, Resistor_SMD:R_0603_1608Metric_Pad0.98x0.95mm_HandSolder, symbol Device:R
- added SW2: ~, LinKey_Lib_Footprints:B3U-1000P, symbol Switch:SW_Omron_B3FS
- added U1: ACPL-214-500E, Package_SO:SOP-4_4.4x2.6mm_P1.27mm, symbol Isolator:ACPL-214-500E
- added U2: ESP32-WROOM-32E, RF_Module:ESP32-WROOM-32E, symbol RF_Module:ESP32-WROOM-32E
- added U4: TL431DBZ, Package_TO_SOT_SMD:SOT-23, symbol Reference_Voltage:TL431DBZ
- added U5: TPS61022, Package_DFN_QFN:Texas_RWU0007A_VQFN-7_2x2mm_P0.5mm, symbol Converter_DCDC:TPS61022
- J1: value (none) -> ~
Connections:
- net at J1.1 (A): now also D1.3 (~_2), R1.2, R3.1
- net at J1.2 (I2): now also D1.2 (~_1), R1.1, R2.1, U1.2
- net at J1.3 (I1): now also R4.1
- new net: R14.1, U4.1 (K)
- new net: R15.2, R16.1, U4.2 (REF)
- new net: R4.2, U1.1
- new net: SW2.1, U2.25 (IO0)
- new net: R7.2, U2.3 (EN)
- new net: D8.4 (BA), R9.1
- new net: D8.5 (GA), R8.1
- new net: L1.2, U5.2 (SW)
- new net: C5.2, R17.2, R18.1, U5.4 (FB)
- new net: Q1.1 (B), R11.2, R14.2
- new net: Q1.3 (C), R12.2, R13.2
- new net: Q2.4 (G), R12.1
- new net: D8.6 (RA), R6.1
- new net: Q2.5 (S), R10.2, R11.1
- new net +3.3V: C5.1, C6.1, C7.1, C8.1, J2.1 (Pin_1), R17.1, R5.2, R7.1, U2.2 (VDD), U5.3 (VOUT)
- new net ESP_RX: J2.3 (Pin_3), U2.34 (RXD0/IO3)
- new net ESP_TX: J2.2 (Pin_2), U2.35 (TXD0/IO1)
- new net GND: C1.2, C2.2, C3.2, C4.2, C6.2, C7.2, C8.2, D1.1 (-), D8.1 (RK), D8.2 (GK), D8.3 (BK), J2.4 (Pin_4), R16.2, R18.2, R2.2, R3.2, SW2.2, U1.3, U2.1 (GND), U2.15 (GND), U2.38 (GND), U2.39 (GND), U4.3 (A), U5.1 (GND), U5.6 (MODE)
- new net LED_BLUE: R6.2, U2.24 (IO2)
- new net LED_GREEN: R9.2, U2.23 (IO15)
- new net LED_RED: R8.2, U2.16 (IO13)
- new net TIC: R5.1, U1.4, U2.13 (IO14)
- new net VCAP: C2.1, C3.1, C4.1, L1.1, Q2.1 (D), Q2.2 (D), Q2.3 (D), R13.1, R15.1, U2.9 (IO33), U5.5 (EN), U5.7 (VIN)
- new net VDD: C1.1, D1.4 (+), Q1.2 (E), R10.1
Other:
- note added: "Icharge=0,7V/R10=39mA"
- note added: "Super Capa"
- note added: "Tcharge=1min30"
- note added: "Umax=2,5V*(R15+R16)/R16=2,7V"
- title: (none) -> Linkey PCB
- moved on the sheet: J1

Commit message: Update pcb version to v1.1
- Fix R10 footprint (was 1206 but should be 0805), decrease value to increase max current to 40mA
- Change R15/R16 values (divided by 10)
- Increase R11 from 200r to 1k to fix voltage limitation
- Fix I1/I2 swap
- Modify R4, R5 values around opto
- Add SW + Capa on EN
Parts:
- added C9: 100n, Capacitor_SMD:C_0603_1608Metric_Pad1.08x0.95mm_HandSolder, symbol Device:C
- added SW1: ~, LinKey_Lib_Footprints:B3U-1000P, symbol Switch:SW_Omron_B3FS
- R10: value 18r -> 10r; footprint Resistor_SMD:R_1206_3216Metric_Pad1.30x1.75mm_HandSolder -> Resistor_SMD:R_0805_2012Metric_Pad1.20x1.40mm_HandSolder; Manufacturer_Part_Number CRCW080518R0FKEA -> CRCW080510R0FKEA; Supplier1_Part_Number 71-CRCW080518R0FKEA -> 71-CRCW0805-10-E3
- R11: value 200r -> 1k; Manufacturer_Part_Number CRCW0603200RFKEAC -> CRCW06031K00FKEAC; Supplier1_Part_Number 71-CRCW0603200RFKEAC -> 71-CRCW06031K00FKEAC
- R15, R5: value 10k -> 1k; Manufacturer_Part_Number CRCW060310K0FKECC -> CRCW06031K00FKEAC; Supplier1_Part_Number 71-CRCW060310K0FKECC -> 71-CRCW06031K00FKEAC
- R16: value 100k -> 10k; Manufacturer_Part_Number CRCW0603100KFKEAC -> CRCW060310K0FKECC; Supplier1_Part_Number 71-CRCW0603100KFKEAC -> 71-CRCW060310K0FKECC
- R4: value 470r -> 330r; Manufacturer_Part_Number CRCW0603470RFKEBC -> CRCW0603330RFKEAC; Supplier1_Part_Number 71-CRCW0603470RFKEBC -> 71-CRCW0603330RFKEAC
Connections:
- net GND: now also C9.2, SW1.1
- net at D1.2 (~_1), R1.1, R2.1: now also J1.3 (I1), R4.1; no longer J1.2 (I2), U1.2
- net at R7.2, U2.3 (EN): now also C9.1, SW1.2
- new net: J1.2 (I2), U1.2
Other:
- moved on the sheet: C1, C7, C8, D1, D8, J1, J2, R1, R2, R3, R4, R5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

Commit message: Update R11 position and J1's 3D model
- Slightly move R11 away from the PCB edge
- Add J1's 3D model
- Complete J1's BOM data = Samtech vertical header that must be manually bent
Parts:
- J1: Manufacturer_Name (none) -> Samtec; Manufacturer_Part_Number (none) -> HPM-03-04-T-S; Supplier1_Name (none) -> Mouser; Supplier1_Part_Number (none) -> 200-HPM0304TS
Changed lines of the file:
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@@
 			)
 		)
-		(property "Description" "Generic connector, single row, 01x04, script generated (kicad-library-utils/schlib/autogen/connector/)"
+		(property "Description" "Headers & Wire Housings .200 Power Terminal Strip"
 			(at 237.49 41.91 0)
 			(effects
@@
 			)
 		)
-		(property "Datasheet" "~"
+		(property "Datasheet" "https://suddendocs.samtec.com/catalog_english/hpm.pdf?_gl=1*mr8nsh*_up*MQ..*_ga*NTc2NzY4MDc5LjE3NDAyMzU5NjI.*_ga_3KFNZC07WW*czE3NzU1OTQ0MDckbzIkZzAkdDE3NzU1OTQ0MDckajYwJGwwJGg2MDEyMTQ0MzQ."
 			(at 67.31 31.75 0)
 			(effects
@@
 			(at 67.31 31.75 0)
 			(effects
+				(font
+					(size 1.27 1.27)
+				)
+				(hide yes)
+			)
+		)
+		(property "Manufacturer_Name" "Samtec"
+			(at 67.31 31.75 0)
+			(effects
+				(font
+					(size 1.27 1.27)
+				)
+				(hide yes)
+			)
+		)
+		(property "Manufacturer_Part_Number" "HPM-03-04-T-S "
+			(at 67.31 31.75 0)
+			(effects
+				(font
+					(size 1.27 1.27)
+				)
+				(hide yes)
+			)
+		)
+		(property "Supplier1_Name" "Mouser"
+			(at 67.31 31.75 0)
+			(effects
+				(font
+					(size 1.27 1.27)
+				)
+				(hide yes)
+			)
+		)
+		(property "Supplier1_Part_Number" "200-HPM0304TS "
+			(at 67.31 31.75 0)
+			(effects
