File: PCB/LinKey.kicad_sch (KiCad schematic)
At the start: 40 parts, among them J2 Conn_01x04, Q1 MMBT2907ALT1G, Q2 CSD25402Q3A, U1 ACPL-214-500E, U2 ESP32-WROOM-32E, U4 TL431DBZ, U5 TPS61022

Commit message: Corrections mineures : - valeur C5 : 15 pF -> 180 pF cohérente avec la référence composant - tension R10 : 75 V -> 150 V cohérente avec la référence composant
Parts:
- C5: value 175p -> 180p
- R10: Voltage 75V -> 150V
Other:
- note added: "Icharge env.= 0,7V/R10"
- note removed: "Icharge=0,7V/R10=39mA"
Changed lines of the file:
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@@
 		(rev "1.1")
 	)
-	(text "Icharge=0,7V/R10=39mA"
+	(text "Icharge env.= 0,7V/R10"
 		(exclude_from_sim no)
 		(at 81.534 115.316 0)
@@
 		)
 		(instances
-			(project ""
+			(project "LinKey"
 				(path "/3bf5bc74-5075-4135-ab8d-3c2b05f42fe2"
 					(reference "R1")
@@
 		)
 		(instances
-			(project ""
+			(project "LinKey"
 				(path "/3bf5bc74-5075-4135-ab8d-3c2b05f42fe2"
 					(reference "R4")
@@
 		)
 		(instances
-			(project ""
+			(project "LinKey"
 				(path "/3bf5bc74-5075-4135-ab8d-3c2b05f42fe2"
 					(reference "R9")
@@
 		)
 		(instances
-			(project ""
+			(project "LinKey"
 				(path "/3bf5bc74-5075-4135-ab8d-3c2b05f42fe2"
 					(reference "R8")
@@
 		)
 		(instances
-			(project ""
+			(project "LinKey"
 				(path "/3bf5bc74-5075-4135-ab8d-3c2b05f42fe2"
 					(reference "U1")
@@
 		)
 		(instances
-			(project ""
+			(project "LinKey"
 				(path "/3bf5bc74-5075-4135-ab8d-3c2b05f42fe2"
 					(reference "#PWR02")
@@
 		)
 		(instances
-			(project ""
+			(project "LinKey"
 				(path "/3bf5bc74-5075-4135-ab8d-3c2b05f42fe2"
 					(reference "J1")
@@
 		)
 		(instances
-			(project ""
+			(project "LinKey"
 				(path "/3bf5bc74-5075-4135-ab8d-3c2b05f42fe2"
 					(reference "R6")
@@
 		)
 		(instances
-			(project ""
+			(project "LinKey"
 				(path "/3bf5bc74-5075-4135-ab8d-3c2b05f42fe2"
 					(reference "#PWR01")
@@
 			)
 		)
-		(property "Voltage" "75V"
+		(property "Voltage" "150V"
 			(at 81.28 111.76 90)
 			(effects
@@
 		)
 		(instances
-			(project ""
+			(project "LinKey"
 				(path "/3bf5bc74-5075-4135-ab8d-3c2b05f42fe2"
 					(reference "#PWR04")
@@
 			)
 		)
-		(property "Value" "175p"
+		(property "Value" "180p"
 			(at 223.52 122.936 0)
 			(effects
