File: PCB/LinKey.kicad_pcb (KiCad board)
At the start: 4 copper layers, 25 x 37.3 mm, 42 parts, among them J2 Conn_01x04, Q1 MMBT2907ALT1G, Q2 CSD25402Q3A, U1 ACPL-214-500E, U2 ESP32-WROOM-32E, U4 TL431DBZ, U5 TPS61022

Commit message: PCB : Modification du modèle 3D et de la position de C2 (supercapa). Couchée orientée pour ne pas interférer avec  les autres composants.
Parts:
- C5: value 175p -> 180p
Changed lines of the file:
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@@
 		)
 		(embedded_fonts no)
-		(model "${KICAD9_3DMODEL_DIR}/Capacitor_THT.3dshapes/CP_Radial_D8.0mm_P3.50mm.step"
+		(model "${KIPRJMOD}/MCAD files/3D step files/Capacitor_THT-CP_Radial_D8.0mm_P3.50mm_special_position - Capacitor_THT-CP_Radial_D8.0mm_P3.50mm_special_position.step"
 			(offset
-				(xyz 0 0 0)
+				(xyz 3.3 2.9 4.5)
 			)
 			(scale
@@
 			)
 			(rotate
-				(xyz 0 0 0)
+				(xyz -0 -0 -155)
 			)
 		)
@@
 			)
 		)
-		(property "Voltage" "75V"
+		(property "Voltage" "150V"
 			(at 0 0 0)
 			(unlocked yes)
@@
 			)
 		)
-		(property "Value" "175p"
+		(property "Value" "180p"
 			(at 0 -1.43 90)
 			(layer "B.Fab")
